File: SigmaLink-USBi.kicad_pcb (KiCad board)
At the start: 2 copper layers, 64 x 39 mm, 36 parts, among them J1 USB_B, J2 Program, J3 Target, U1 LM1117-3.3, U2 24LC512, U3 CY7C68013A-56, U4 MAX809, U5 74LVC2G66, U6 TPS2051B, Y1 24MHz

Commit message: Rerouted the board
Parts:
- removed R1: 10k, Resistors_SMD:R_0603_HandSoldering
- added D4: PRTR5V0U2X, Package_TO_SOT_SMD:SOT-143, F.Cu at (130.3, 84.8)
- added RN2: 4.7k, Resistor_SMD:R_Array_Convex_4x0603, F.Cu at (164.6, 101.9)
- added RN3: 22, Resistor_SMD:R_Array_Convex_4x0603, F.Cu at (134.8, 91.1)
- C1, C2: footprint Capacitors_SMD:CP_Elec_6.3x5.3 -> Capacitor_SMD:CP_Elec_6.3x5.3
- C10, C11, C12, C13, C3, C4, C5, C6, C7, C8, C9: footprint Capacitors_SMD:C_0603_HandSoldering -> Capacitor_SMD:C_0603_1608Metric_Pad1.05x0.95mm_HandSolder
- D1, D3: footprint LEDs:LED-3MM -> LED_THT:LED_D3.0mm
- D2: footprint LEDs:LED_D3.0mm-3 -> LED_THT:LED_D3.0mm-3
- F1: footprint Resistors_SMD:R_0805_HandSoldering -> Fuse:Fuse_1812_4532Metric_Pad1.30x3.40mm_HandSolder
- J1: footprint Connectors:USB_B -> Connector_USB:USB_B_OST_USB-B1HSxx_Horizontal
- J2: footprint Pin_Headers:Pin_Header_Straight_1x02_Pitch2.54mm -> Connector_PinHeader_1.27mm:PinHeader_2x01_P1.27mm_Vertical
- J3: footprint Connectors_Multicomp:Multicomp_MC9A22-1434_2x07x2.54mm_Angled -> Connector_IDC:IDC-Header_2x07_P2.54mm_Horizontal
- R2, R3, R4, R5, R6, R7, R8: footprint Resistors_SMD:R_0603_HandSoldering -> Resistor_SMD:R_0603_1608Metric_Pad1.05x0.95mm_HandSolder
- RN1: footprint Resistors_SMD:R_Array_Convex_4x0603 -> Resistor_SMD:R_Array_Convex_4x0603
- U1: footprint TO_SOT_Packages_SMD:SOT-223-3Lead_TabPin2 -> Package_TO_SOT_SMD:SOT-223-3_TabPin2
- U2: footprint Housings_SOIC:SOIC-8_3.9x4.9mm_Pitch1.27mm -> Package_SO:SOIC-8_3.9x4.9mm_P1.27mm
- U3: footprint CY7C68013:QFN56_8x8mm -> Package_DFN_QFN:QFN-56-1EP_8x8mm_P0.5mm_EP4.6x5.3mm
- U4: footprint TO_SOT_Packages_SMD:SOT-23_Handsoldering -> Package_TO_SOT_SMD:SOT-23W
- U5: footprint Housings_SSOP:VSSOP-8_2.3x2mm_Pitch0.5mm -> Package_SO:VSSOP-8_2.3x2mm_P0.5mm
- U6: footprint TO_SOT_Packages_SMD:SOT-23-5_HandSoldering -> Package_TO_SOT_SMD:SOT-23-5
- Y1: footprint Crystals:Crystal_SMD_5032-2pin_5.0x3.2mm_HandSoldering -> Crystal:Crystal_SMD_5032-2Pin_5.0x3.2mm_HandSoldering
- moved J2 25.7 mm to (165.2, 98.7), turned to 180 degrees
- moved R6 16.3 mm to (164.6, 89.8), turned to 180 degrees
- moved U2 12.9 mm to (158.9, 100.6), turned to 180 degrees
- moved C12 5.43 mm to (150.0, 86.0), turned to 90 degrees
- moved F1 1.91 mm to (121.4, 110.2)
- moved C6 1.80 mm to (143.7, 89.2), turned to 90 degrees
- moved C8 1.27 mm to (143.7, 99.4), turned to 0 degrees
- moved D1 0.63 mm to (160.2, 113.3)
- moved D2 0.63 mm to (150.0, 112.1)
- moved D3 0.63 mm to (139.8, 113.3)
- turned J3 to 0 degrees
Connections:
- J1 pad 2: /D- -> /UD-
- J1 pad 3: /D+ -> /UD+
- U2 pad 1: +3V3 -> Net-(RN2-Pad7)
- U2 pad 2: GND -> Net-(RN2-Pad6)
- U2 pad 3: GND -> Net-(RN2-Pad5)
Routing:
- net +5V: track 50.0 -> 89.0 mm
- net /TMCLK: track 50.4 -> 15.2 mm
- net GND: track 32.4 -> 8.54 mm, vias 11 -> 253
- net /UD-: track 0.00 -> 20.1 mm, vias 0 -> 2
- net /UD+: track 0.00 -> 19.8 mm, vias 0 -> 2
- net /SCL: track 21.1 -> 33.5 mm, vias 2 -> 3
- net /MCK: track 5.04 -> 17.3 mm, vias 0 -> 2
- net /D-: track 20.9 -> 11.9 mm
- net /D+: track 20.8 -> 11.9 mm
- net /SDA: track 23.5 -> 31.0 mm, vias 2 -> 3
- net /TRESET: track 58.4 -> 51.7 mm
- net /TSCL: track 26.3 -> 32.8 mm
- net /~TLATCH1: track 40.5 -> 46.3 mm
- net +3V3: track 137.9 -> 132.1 mm, vias 10 -> 16
- net /~TLATCH4: track 26.5 -> 32.2 mm, vias 2 -> 1
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Other:
- outline, holes or cut-outs redrawn
