File: SigmaLink-USBi.kicad_pcb (KiCad board)
At the start: 2 copper layers, 64 x 39 mm, 30 parts, among them J1 USB_B, J2 Program, J3 Target, U1 LM1117-3.3, U2 24LC512, U3 CY7C68013A-56, U4 MAX809, U5 74LVC2G66, U6 TPS2051B, Y1 24MHz

Commit message: General maintanence commit.
Parts:
- added D4: B5819W, Diode_SMD:D_SOD-123, F.Cu at (164.6, 108.9)
- J2: footprint Connector_PinHeader_1.27mm:PinHeader_2x01_P1.27mm_Vertical -> Connector_PinHeader_1.27mm:PinHeader_1x02_P1.27mm_Vertical
- Y1: footprint Crystal:Crystal_SMD_5032-2Pin_5.0x3.2mm -> Crystal:Crystal_HC49-4H_Vertical
- moved C4 3.86 mm to (131.6, 83.5)
- moved C3 1.42 mm to (139.2, 83.5)
- moved C5 0.64 mm to (157.0, 87.9)
- moved R6 0.64 mm to (157.0, 86.0)
- moved R7 0.64 mm to (157.0, 90.5)
- moved U4 0.63 mm to (160.8, 89.2)
- turned J2 to 270 degrees
Connections:
- C11 pad 1: +3V3 -> Net-(C11-Pad1)
- RN2 pad 1: +3V3 -> Net-(C11-Pad1)
- RN2 pad 2: +3V3 -> Net-(C11-Pad1)
- RN4 pad 1: (no net) -> Net-(C11-Pad1)
- RN4 pad 5: +3V3 -> Net-(C11-Pad1)
- RN4 pad 6: +3V3 -> Net-(C11-Pad1)
- RN4 pad 7: +3V3 -> Net-(C11-Pad1)
- RN4 pad 8: +3V3 -> Net-(C11-Pad1)
- U2 pad 8: +3V3 -> Net-(C11-Pad1)
Routing:
- net Net-(C11-Pad1): track 0.00 -> 30.0 mm, vias 0 -> 3
- net +3V3: track 131.8 -> 115.7 mm, vias 15 -> 11
- net /XTALO: track 15.4 -> 17.8 mm
- net /LED_SPI: track 13.8 -> 14.5 mm, vias 2 -> 0
- net /MCK: track 9.57 -> 10.2 mm
- net Net-(R7-Pad2): track 1.67 -> 2.31 mm
- net /TMCLK: track 27.7 -> 27.1 mm
- net /XTALI: track 18.7 -> 19.3 mm
- net GND: vias 558 -> 516
- net (no net): vias 0 -> 1
Other:
- board text added: "SigmaLink USBi © 2019 Max Chan"
- board text removed: "SigmaLink USBi © 2018 Max Chan"
