File: SigmaLink-USBi.sch (KiCad schematic (older format))
At the start: 36 parts, among them J1 USB_B, J2 Program, J3 Target, U1 LM1117-3.3, U2 24LC512, U3 CY7C68013A-56, U4 MAX809, U5 74LVC2G66, U6 TPS2051B, Y1 24MHz

Commit message: Preparing for v1r2
Parts:
- removed R1: 10k, Resistors_SMD:R_0603_HandSoldering, symbol R_Small
- added D?: PRTR5V0U2X, symbol Power_Protection:PRTR5V0U2X
- added RN?: 4.7k, symbol Device:R_Pack04
- added RN?: 22, symbol Device:R_Pack04
- C1, C2: symbol CP_Small -> Device:CP_Small
- C10, C11, C12, C13, C3, C4, C5, C6, C7, C8, C9: symbol C_Small -> Device:C_Small
- D1, D3: symbol LED -> Device:LED
- D2: symbol LED_Dual_CAC -> Device:LED_Dual_CAC
- F1: symbol Polyfuse_Small -> Device:Polyfuse_Small
- J1: symbol USB_B -> SigmaLink-USBi-rescue:USB_B
- J2: symbol GS2 -> SigmaLink-USBi-rescue:GS2
- J3: symbol Conn_02x07_Odd_Even -> SigmaLink-USBi-rescue:Conn_02x07_Odd_Even
- R2, R3, R4, R5, R6, R7, R8: symbol R_Small -> Device:R_Small
- RN1: symbol R_Pack04 -> Device:R_Pack04
- U1: symbol LM1117-3.3 -> SigmaLink-USBi-rescue:LM1117-3.3
- U2: symbol 24LC512 -> SigmaLink-USBi-rescue:24LC512
- U3: symbol CY7C68013A-56 -> cy7c68013:CY7C68013A-56
- U4: symbol MAX809 -> usb-mux:MAX809
- U5: symbol 74LVC2G66 -> 74xGxx:74LVC2G66
- U6: symbol TPS2051B -> SigmaLink-USBi-rescue:TPS2051B
- Y1: symbol Crystal_Small -> Device:Crystal_Small
Connections:
- net labels added: UD+, UD-
- wire segments 157 -> 242
Other:
- moved on the sheet: J1, J2, U1, U2

Commit message: Rerouted the board
Parts:
- C1, C2: footprint Capacitors_SMD:CP_Elec_6.3x5.3 -> Capacitor_SMD:CP_Elec_6.3x5.3
- C10, C11, C12, C13, C3, C4, C5, C6, C7, C8, C9: footprint Capacitors_SMD:C_0603_HandSoldering -> Capacitor_SMD:C_0603_1608Metric_Pad1.05x0.95mm_HandSolder
- D1, D3: footprint LEDs:LED-3MM -> LED_THT:LED_D3.0mm
- D2: footprint LEDs:LED_D3.0mm-3 -> LED_THT:LED_D3.0mm-3
- D4: renamed from D?; footprint (none) -> Package_TO_SOT_SMD:SOT-143
- F1: footprint Resistors_SMD:R_0805_HandSoldering -> Fuse:Fuse_1812_4532Metric_Pad1.30x3.40mm_HandSolder
- J1: footprint Connectors:USB_B -> Connector_USB:USB_B_OST_USB-B1HSxx_Horizontal
- J2: footprint Pin_Headers:Pin_Header_Straight_1x02_Pitch2.54mm -> Connector_PinHeader_1.27mm:PinHeader_2x01_P1.27mm_Vertical
- J3: footprint Connectors_Multicomp:Multicomp_MC9A22-1434_2x07x2.54mm_Angled -> Connector_IDC:IDC-Header_2x07_P2.54mm_Horizontal
- R2, R3, R4, R5, R6, R7, R8: footprint Resistors_SMD:R_0603_HandSoldering -> Resistor_SMD:R_0603_1608Metric_Pad1.05x0.95mm_HandSolder
- RN1: footprint Resistors_SMD:R_Array_Convex_4x0603 -> Resistor_SMD:R_Array_Convex_4x0603
- RN2, RN3: renamed from RN?; footprint (none) -> Resistor_SMD:R_Array_Convex_4x0603
- U1: footprint TO_SOT_Packages_SMD:SOT-223-3Lead_TabPin2 -> Package_TO_SOT_SMD:SOT-223-3_TabPin2
- U2: footprint Housings_SOIC:SOIC-8_3.9x4.9mm_Pitch1.27mm -> Package_SO:SOIC-8_3.9x4.9mm_P1.27mm
- U3: footprint CY7C68013:QFN56_8x8mm -> Package_DFN_QFN:QFN-56-1EP_8x8mm_P0.5mm_EP4.6x5.3mm
- U4: footprint TO_SOT_Packages_SMD:SOT-23_Handsoldering -> Package_TO_SOT_SMD:SOT-23W
- U5: footprint Housings_SSOP:VSSOP-8_2.3x2mm_Pitch0.5mm -> Package_SO:VSSOP-8_2.3x2mm_P0.5mm
- U6: footprint TO_SOT_Packages_SMD:SOT-23-5_HandSoldering -> Package_TO_SOT_SMD:SOT-23-5
- Y1: footprint Crystals:Crystal_SMD_5032-2pin_5.0x3.2mm_HandSoldering -> Crystal:Crystal_SMD_5032-2Pin_5.0x3.2mm_HandSoldering
