File: SigmaLink-USBi.sch (KiCad schematic (older format))
At the start: 38 parts, among them J1 USB_B, J2 Program, J3 Target, U1 LM1117-3.3, U2 24LC512, U3 CY7C68013A-56, U4 MAX809, U5 74LVC2G66, U6 TPS2051B, Y1 24MHz

Commit message: Resistor packs are used more extensively.
Also a re-layout.
Parts:
- removed C10, C12, C8: 100n, Capacitor_SMD:C_0603_1608Metric_Pad1.05x0.95mm_HandSolder, symbol Device:C_Small
- removed D4: PRTR5V0U2X, Package_TO_SOT_SMD:SOT-143, symbol Power_Protection:PRTR5V0U2X
- removed R2, R3: 4.7k, Resistor_SMD:R_0603_1608Metric_Pad1.05x0.95mm_HandSolder, symbol Device:R_Small
- removed R4, R5, R8: 10k, Resistor_SMD:R_0603_1608Metric_Pad1.05x0.95mm_HandSolder, symbol Device:R_Small
- added RN4: 4.7k, Resistor_SMD:R_Array_Convex_4x0603, symbol Device:R_Pack04
- J3: symbol SigmaLink-USBi-rescue:Conn_02x07_Odd_Even -> Connector_Generic:Conn_02x07_Odd_Even
- RN3: value 22 -> 10k
- U4: footprint Package_TO_SOT_SMD:SOT-23W -> Package_TO_SOT_SMD:SOT-23
- U5: footprint Package_SO:VSSOP-8_2.3x2mm_P0.5mm -> Package_SO:VSSOP-8_3.0x3.0mm_P0.65mm
- Y1: footprint Crystal:Crystal_SMD_5032-2Pin_5.0x3.2mm_HandSoldering -> Crystal:Crystal_SMD_5032-2Pin_5.0x3.2mm
Connections:
- net labels removed: UD+, UD-
- wire segments 242 -> 224
- no-connect marks 23 -> 22
Other:
- moved on the sheet: C1, C11, C13, C2, C3, C4, C5, C6, C7, C9, D1, D2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
